File: sheet_heart.sch (KiCad schematic (older format))
At the start: 41 parts, among them P1 CONN_02X05, P7 CONN_01X01, P8 CONN_01X01, U4 STM32F042GxU

Commit message: Change RGB LED footprint to match new batch of cheap 0603.
Parts:
- LD7: footprint knielsenlib:RGB_0603 -> knielsenlib:RGB_0603_ALTPINOUT
Changed lines of the file:
@@
 F 0 "LD7" H 8900 5041 40  0000 C CNN
 F 1 "RGB" H 8900 4965 40  0000 C CNN
-F 2 "knielsenlib:RGB_0603" H 8375 4875 60  0001 C CNN
+F 2 "knielsenlib:RGB_0603_ALTPINOUT" H 8375 4875 60  0001 C CNN
 F 3 "" H 8375 4875 60  0000 C CNN
 	1    8900 4800
